Commit message: Strap robot model down to differential wheelbase

File: goldorak_simulation/urdf/goldorak.xacro (robot description, xacro)
@@ -1,10 +1,10 @@
 <?xml version="1.0"?>
 <robot name="goldorak" xmlns:xacro="http://ros.org/wiki/xacro">
-  <xacro:property name="width" value=".2" />
-  <xacro:property name="leglen" value=".6" />
-  <xacro:property name="polelen" value=".2" />
-  <xacro:property name="bodylen" value=".6" />
-  <xacro:property name="baselen" value=".4" />
-  <xacro:property name="wheeldiam" value=".07" />
+  <xacro:property name="body_width" value="0.2" />
+  <xacro:property name="body_height" value="0.1" />
+  <xacro:property name="wheelbase" value="0.3" />
+  <xacro:property name="wheel_diameter" value="0.1" />
+  <xacro:property name="wheel_thickness" value="0.1" />
+  <xacro:property name="wheel_offset" value="0.05" />
   <xacro:property name="pi" value="3.1415" />
   <material name="blue">
@@ -26,21 +26,21 @@
     <visual>
       <geometry>
-        <cylinder radius="${width}" length="${bodylen}"/>
+        <cylinder radius="${body_width}" length="${body_height}"/>
       </geometry>
-      <material name="blue"/>
+      <material name="white"/>
     </visual>
     <collision>
       <geometry>
-        <cylinder radius="${width}" length="${bodylen}"/>
+        <cylinder radius="${body_width}" length="${body_height}"/>
       </geometry>
     </collision>
     <xacro:default_inertial mass="10"/>
   </link>
-  <xacro:macro name="wheel" params="prefix suffix reflect">
-    <link name="${prefix}_${suffix}_wheel">
+  <xacro:macro name="wheel" params="prefix reflect">
+    <link name="${prefix}_wheel">
       <visual>
         <origin xyz="0 0 0" rpy="${pi/2} 0 0" />
         <geometry>
-          <cylinder radius="${wheeldiam/2}" length="0.1"/>
+          <cylinder radius="${wheel_diameter/2}" length="0.01"/>
         </geometry>
         <material name="black"/>
@@ -50,5 +50,5 @@
         <origin xyz="0 0 0" rpy="${pi/2} 0 0" />
         <geometry>
-          <cylinder radius="${wheeldiam/2}" length="0.1"/>
+          <cylinder radius="${wheel_diameter/2}" length="${wheel_thickness}"/>
         </geometry>
         <origin xyz="0 0 0" rpy="0 0 0" />
@@ -56,13 +56,16 @@
       <xacro:default_inertial mass="1"/>
     </link>
-    <joint name="${prefix}_${suffix}_wheel_joint" type="continuous">
+    <joint name="${prefix}_wheel_joint" type="continuous">
       <axis xyz="0 1 0" rpy="0 0 0" />
-      <parent link="${prefix}_base"/>
-      <child link="${prefix}_${suffix}_wheel"/>
-      <origin xyz="${baselen*reflect/3} 0 -${wheeldiam/2+.05}" rpy="0 0 0"/>
+      <parent link="base_link"/>
+      <child link="${prefix}_wheel"/>
+      <origin xyz="0
+                   ${(wheelbase + wheel_thickness) * reflect / 2}
+                   -${wheel_diameter / 2 - wheel_offset}"
+              rpy="0 0 0"/>
     </joint>
     <!-- This block provides the simulator (Gazebo) with information on a few additional
     physical properties. See http://gazebosim.org/tutorials/?tut=ros_urdf for more-->
-    <gazebo reference="${prefix}_${suffix}_wheel">
+    <gazebo reference="${prefix}_wheel">
       <mu1 value="200.0"/>
       <mu2 value="100.0"/>
@@ -73,201 +76,16 @@
     <!-- This block connects the wheel joint to an actuator (motor), which informs both
     simulation and visualization of the robot -->
-    <transmission name="${prefix}_${suffix}_wheel_trans" type="SimpleTransmission">
+    <transmission name="${prefix}_wheel_trans" type="SimpleTransmission">
       <type>transmission_interface/SimpleTransmission</type>
-      <actuator name="${prefix}_${suffix}_wheel_motor">
+      <actuator name="${prefix}_wheel_motor">
         <mechanicalReduction>1</mechanicalReduction>
       </actuator>
-      <joint name="${prefix}_${suffix}_wheel_joint">
+      <joint name="${prefix}_wheel_joint">
         <hardwareInterface>VelocityJointInterface</hardwareInterface>
       </joint>
     </transmission>
   </xacro:macro>
-  <xacro:macro name="leg" params="prefix reflect">
-    <link name="${prefix}_leg">
-      <visual>
-        <geometry>
-          <box size="${leglen} .1 .2"/>
-        </geometry>
-        <origin xyz="0 0 -${leglen/2}" rpy="0 ${pi/2} 0"/>
-        <material name="white"/>
-      </visual>
-      <collision>
-        <geometry>
-          <box size="${leglen} .1 .2"/>
-        </geometry>
-        <origin xyz="0 0 -${leglen/2}" rpy="0 ${pi/2} 0"/>
-      </collision>
-      <xacro:default_inertial mass="10"/>
-    </link>
-    <joint name="base_to_${prefix}_leg" type="fixed">
-      <parent link="base_link"/>
-      <child link="${prefix}_leg"/>
-      <origin xyz="0 ${reflect*(width+.02)} .25" />
-    </joint>
-    <link name="${prefix}_base">
-      <visual>
-        <geometry>
-          <box size="${baselen} .1 .1"/>
-        </geometry>
-        <material name="white"/>
-      </visual>
-      <collision>
-        <geometry>
-          <box size="${baselen} .1 .1"/>
-        </geometry>
-      </collision>
-      <xacro:default_inertial mass="10"/>
-    </link>
-    <joint name="${prefix}_base_joint" type="fixed">
-      <parent link="${prefix}_leg"/>
-      <child link="${prefix}_base"/>
-      <origin xyz="0 0 ${-leglen}" />
-    </joint>
-    <xacro:wheel prefix="${prefix}" suffix="front" reflect="1"/>
-    <xacro:wheel prefix="${prefix}" suffix="back" reflect="-1"/>
-  </xacro:macro>
-  <xacro:leg prefix="right" reflect="-1" />
-  <xacro:leg prefix="left" reflect="1" />
-  <joint name="gripper_extension" type="prismatic">
-    <parent link="base_link"/>
-    <child link="gripper_pole"/>
-    <limit effort="1000.0" lower="-${width*2-.02}" upper="0" velocity="0.5"/>
-    <origin rpy="0 0 0" xyz="${width-.01} 0 .2"/>
-    <limit effort="30" velocity="0.2"/>
-    <dynamics damping="0.0" friction="0.0"/>
-  </joint>
-  <link name="gripper_pole">
-    <visual>
-      <geometry>
-        <cylinder length="${polelen}" radius=".01"/>
-      </geometry>
-      <origin xyz="${polelen/2} 0 0" rpy="0 ${pi/2} 0 "/>
-    </visual>
-    <collision>
-      <geometry>
-        <cylinder length="${polelen}" radius=".01"/>
-      </geometry>
-      <origin xyz="${polelen/2} 0 0" rpy="0 ${pi/2} 0 "/>
-    </collision>
-    <xacro:default_inertial mass=".05"/>
-  </link>
-  <transmission name="gripper_extension_trans" type="SimpleTransmission">
-    <type>transmission_interface/SimpleTransmission</type>
-    <actuator name="gripper_extension_motor">
-      <mechanicalReduction>1</mechanicalReduction>
-    </actuator>
-    <joint name="gripper_extension">
-      <hardwareInterface>PositionJointInterface</hardwareInterface>
-    </joint>
-  </transmission>
-  <xacro:macro name="gripper" params="prefix reflect">
-    <joint name="${prefix}_gripper_joint" type="revolute">
-      <axis xyz="0 0 ${reflect}"/>
-      <limit effort="1000.0" lower="0.0" upper="0.548" velocity="0.5"/>
-      <origin rpy="0 0 0" xyz="${polelen} ${reflect*0.01} 0"/>
-      <parent link="gripper_pole"/>
-      <child link="${prefix}_gripper"/>
-      <limit effort="30" velocity="1.0"/>
-      <dynamics damping="0.0" friction="0.0"/>
-    </joint>
-    <link name="${prefix}_gripper">
-      <visual>
-        <origin rpy="${(reflect-1)/2*pi} 0 0" xyz="0 0 0"/>
-        <geometry>
-          <mesh filename="package://pr2_description/meshes/gripper_v0/l_finger.dae"/>
-        </geometry>
-      </visual>
-      <collision>
-        <geometry>
-          <mesh filename="package://pr2_description/meshes/gripper_v0/l_finger.dae"/>
-        </geometry>
-        <origin rpy="${(reflect-1)/2*pi} 0 0" xyz="0 0 0"/>
-      </collision>
-      <xacro:default_inertial mass=".05"/>
-    </link>
-    <transmission name="${prefix}_gripper_trans" type="SimpleTransmission">
-      <type>transmission_interface/SimpleTransmission</type>
-      <actuator name="${prefix}_gripper_motor">
-        <mechanicalReduction>1</mechanicalReduction>
-      </actuator>
-      <joint name="${prefix}_gripper_joint">
-        <hardwareInterface>PositionJointInterface</hardwareInterface>
-      </joint>
-    </transmission>
-    <joint name="${prefix}_tip_joint" type="fixed">
-      <parent link="${prefix}_gripper"/>
-      <child link="${prefix}_tip"/>
-    </joint>
-    <link name="${prefix}_tip">
-      <visual>
-        <origin rpy="${(reflect-1)/2*pi} 0 0" xyz="0.09137 0.00495 0"/>
-        <geometry>
-          <mesh filename="package://pr2_description/meshes/gripper_v0/l_finger_tip.dae"/>
-        </geometry>
-      </visual>
-      <collision>
-        <geometry>
-          <mesh filename="package://pr2_description/meshes/gripper_v0/l_finger_tip.dae"/>
-        </geometry>
-        <origin rpy="${(reflect-1)/2*pi} 0 0" xyz="0.09137 0.00495 0"/>
-      </collision>
-      <xacro:default_inertial mass=".05"/>
-    </link>
-  </xacro:macro>
-  <xacro:gripper prefix="left" reflect="1" />
-  <xacro:gripper prefix="right" reflect="-1" />
-  <link name="head">
-    <visual>
-      <geometry>
-        <sphere radius="${width}"/>
-      </geometry>
-      <material name="white"/>
-    </visual>
-    <collision>
-      <geometry>
-        <sphere radius="${width}"/>
-      </geometry>
-    </collision>
-    <xacro:default_inertial mass="2"/>
-  </link>
-  <joint name="head_swivel" type="continuous">
-    <parent link="base_link"/>
-    <child link="head"/>
-    <axis xyz="0 0 1"/>
-    <origin xyz="0 0 ${bodylen/2}"/>
-    <limit effort="30" velocity="1.0"/>
-    <dynamics damping="0.0" friction="0.0"/>
-  </joint>
-  <!-- This block connects the head_swivel joint to an actuator (motor), which informs both
-  simulation and visualization of the robot -->
-  <transmission name="head_swivel_trans" type="SimpleTransmission">
-    <type>transmission_interface/SimpleTransmission</type>
-    <actuator name="$head_swivel_motor">
-      <mechanicalReduction>1</mechanicalReduction>
-    </actuator>
-    <joint name="head_swivel">
-      <hardwareInterface>PositionJointInterface</hardwareInterface>
-    </joint>
-  </transmission>
-  <link name="box">
-    <visual>
-      <geometry>
-        <box size=".08 .08 .08"/>
-      </geometry>
-      <material name="blue"/>
-      <origin xyz="-0.04 0 0"/>
-    </visual>
-    <collision>
-      <geometry>
-        <box size=".08 .08 .08"/>
-      </geometry>
-    </collision>
-    <xacro:default_inertial mass="1"/>
-  </link>
-  <joint name="tobox" type="fixed">
-    <parent link="head"/>
-    <child link="box"/>
-    <origin xyz="${.707*width+0.04} 0 ${.707*width}"/>
-  </joint>
+  <xacro:wheel prefix="right" reflect="1"/>
+  <xacro:wheel prefix="left" reflect="-1"/>
   <!-- Gazebo plugin for ROS Control -->
   <gazebo>

Commit message: Add 1D lidar to robot simulation

File: goldorak_simulation/urdf/goldorak.xacro (robot description, xacro)
@@ -88,4 +88,30 @@
   <xacro:wheel prefix="right" reflect="1"/>
   <xacro:wheel prefix="left" reflect="-1"/>
+  <!-- Laser scanner 1D -->
+  <joint name="laser_joint" type="fixed">
+    <axis xyz="0 1 0" />
+    <origin xyz="0 0 ${body_height}" rpy="0 0 0"/>
+    <parent link="base_link"/>
+    <child link="laser_link"/>
+  </joint>
+  <link name="laser_link">
+    <collision>
+      <origin xyz="0 0 0" rpy="0 0 0"/>
+      <geometry>
+        <cylinder radius="0.05" length="0.1"/>
+      </geometry>
+    </collision>
+    <visual>
+      <origin xyz="0 0 0" rpy="0 0 0"/>
+      <geometry>
+        <cylinder radius="0.05" length="0.1"/>
+      </geometry>
+    </visual>
+    <inertial>
+      <mass value="1e-5" />
+      <origin xyz="0 0 0" rpy="0 0 0"/>
+      <inertia ixx="1e-6" ixy="0" ixz="0" iyy="1e-6" iyz="0" izz="1e-6" />
+    </inertial>
+  </link>
   <!-- Gazebo plugin for ROS Control -->
   <gazebo>
@@ -94,3 +120,35 @@
     </plugin>
   </gazebo>
+  <!-- Gazebo plugin for Laser scanner -->
+  <gazebo reference="laser_link">
+    <sensor type="ray" name="laser_sensor">
+      <pose>0 0 0 0 0 0</pose>
+      <visualize>true</visualize>
+      <update_rate>40</update_rate>
+      <ray>
+        <scan>
+          <horizontal>
+            <samples>1</samples>
+            <resolution>1</resolution>
+            <min_angle>-1.570796</min_angle>
+            <max_angle>1.570796</max_angle>
+          </horizontal>
+        </scan>
+        <range>
+          <min>0.10</min>
+          <max>30.0</max>
+          <resolution>0.01</resolution>
+        </range>
+        <noise>
+          <type>gaussian</type>
+          <mean>0.0</mean>
+          <stddev>0.01</stddev>
+        </noise>
+      </ray>
+      <plugin name="gazebo_ros_laser_controller" filename="libgazebo_ros_laser.so">
+        <topicName>/laser/scan</topicName>
+        <frameName>laser_link</frameName>
+      </plugin>
+    </sensor>
+  </gazebo>
 </robot>

Commit message: Publish robot TF using URDF

File: goldorak_simulation/urdf/goldorak.xacro (robot description, xacro)
@@ -5,5 +5,5 @@
   <xacro:property name="wheelbase" value="0.3" />
   <xacro:property name="wheel_diameter" value="0.1" />
-  <xacro:property name="wheel_thickness" value="0.1" />
+  <xacro:property name="wheel_thickness" value="0.01" />
   <xacro:property name="wheel_offset" value="0.05" />
   <xacro:property name="pi" value="3.1415" />
@@ -42,5 +42,5 @@
         <origin xyz="0 0 0" rpy="${pi/2} 0 0" />
         <geometry>
-          <cylinder radius="${wheel_diameter/2}" length="0.01"/>
+          <cylinder radius="${wheel_diameter/2}" length="${wheel_thickness}"/>
         </geometry>
         <material name="black"/>
@@ -57,5 +57,5 @@
     </link>
     <joint name="${prefix}_wheel_joint" type="continuous">
-      <axis xyz="0 1 0" rpy="0 0 0" />
+      <axis xyz="0 ${reflect} 0" rpy="0 0 0" />
       <parent link="base_link"/>
       <child link="${prefix}_wheel"/>

Commit message: Fix oscillation of the robot in simulation
Also scale up the base link

File: goldorak_simulation/urdf/goldorak.xacro (robot description, xacro)
@@ -1,10 +1,13 @@
 <?xml version="1.0"?>
 <robot name="goldorak" xmlns:xacro="http://ros.org/wiki/xacro">
-  <xacro:property name="body_width" value="0.2" />
-  <xacro:property name="body_height" value="0.1" />
-  <xacro:property name="wheelbase" value="0.3" />
-  <xacro:property name="wheel_diameter" value="0.1" />
+  <xacro:property name="body_radius" value="0.12" />
+  <xacro:property name="body_height" value="0.5" />
+  <xacro:property name="wheelbase" value="0.194" />
+  <xacro:property name="wheel_radius" value="0.029" />
   <xacro:property name="wheel_thickness" value="0.01" />
-  <xacro:property name="wheel_offset" value="0.05" />
+  <xacro:property name="wheel_offset" value="-0.20" />
+  <xacro:property name="casterbase" value="0.194" />
+  <xacro:property name="caster_radius" value="0.01" />
+  <xacro:property name="caster_offset" value="-0.24" />
   <xacro:property name="pi" value="3.1415" />
   <material name="blue">
@@ -20,5 +23,7 @@
     <inertial>
       <mass value="${mass}" />
-      <inertia ixx="1.0" ixy="0.0" ixz="0.0" iyy="1.0" iyz="0.0" izz="1.0" />
+      <inertia ixx="1.0" ixy="0.0" ixz="0.0"
+               iyy="1.0" iyz="0.0"
+               izz="1.0" />
     </inertial>
   </xacro:macro>
@@ -26,5 +31,5 @@
     <visual>
       <geometry>
-        <cylinder radius="${body_width}" length="${body_height}"/>
+        <cylinder radius="${body_radius}" length="${body_height}"/>
       </geometry>
       <material name="white"/>
@@ -32,8 +37,14 @@
     <collision>
       <geometry>
-        <cylinder radius="${body_width}" length="${body_height}"/>
+        <cylinder radius="${body_radius}" length="${body_height}"/>
       </geometry>
     </collision>
-    <xacro:default_inertial mass="10"/>
+    <inertial>
+      <mass value="2" />
+      <origin xyz="0 0 0.0" />
+      <inertia ixx="0.01" ixy="0.0" ixz="0.0"
+               iyy="0.01" iyz="0.0"
+               izz="0.5" />
+    </inertial>
   </link>
   <xacro:macro name="wheel" params="prefix reflect">
@@ -42,5 +53,5 @@
         <origin xyz="0 0 0" rpy="${pi/2} 0 0" />
         <geometry>
-          <cylinder radius="${wheel_diameter/2}" length="${wheel_thickness}"/>
+          <cylinder radius="${wheel_radius}" length="${wheel_thickness}"/>
         </geometry>
         <material name="black"/>
@@ -50,17 +61,23 @@
         <origin xyz="0 0 0" rpy="${pi/2} 0 0" />
         <geometry>
-          <cylinder radius="${wheel_diameter/2}" length="${wheel_thickness}"/>
+          <cylinder radius="${wheel_radius}" length="${wheel_thickness}"/>
         </geometry>
         <origin xyz="0 0 0" rpy="0 0 0" />
       </collision>
-      <xacro:default_inertial mass="1"/>
+      <inertial>
+          <origin xyz="0 0 0"/>
+          <mass value="0.01" />
+          <inertia ixx="0.001" ixy="0.0" ixz="0.0"
+                   iyy="0.001" iyz="0.0"
+                   izz="0.001" />
+        </inertial>
     </link>
     <joint name="${prefix}_wheel_joint" type="continuous">
-      <axis xyz="0 ${reflect} 0" rpy="0 0 0" />
+      <axis xyz="0 1 0" rpy="0 0 0" />
       <parent link="base_link"/>
       <child link="${prefix}_wheel"/>
       <origin xyz="0
                    ${(wheelbase + wheel_thickness) * reflect / 2}
-                   -${wheel_diameter / 2 - wheel_offset}"
+                   ${wheel_offset - wheel_radius}"
               rpy="0 0 0"/>
     </joint>
@@ -68,8 +85,8 @@
     physical properties. See http://gazebosim.org/tutorials/?tut=ros_urdf for more-->
     <gazebo reference="${prefix}_wheel">
-      <mu1 value="200.0"/>
-      <mu2 value="100.0"/>
-      <kp value="10000000.0" />
-      <kd value="1.0" />
+      <mu1>1.0</mu1>
+      <mu2>1.0</mu2>
+      <kp>1000000.0</kp>
+      <kd>100.0</kd>
       <material>Gazebo/Grey</material>
     </gazebo>
@@ -88,8 +105,54 @@
   <xacro:wheel prefix="right" reflect="1"/>
   <xacro:wheel prefix="left" reflect="-1"/>
+  <xacro:macro name="caster" params="prefix reflect">
+    <link name="${prefix}_caster">
+      <visual>
+        <origin xyz="0 0 0" rpy="${pi/2} 0 0" />
+        <geometry>
+          <sphere radius="${caster_radius}" />
+        </geometry>
+        <material name="black"/>
+        <origin xyz="0 0 0" rpy="0 0 0" />
+      </visual>
+      <collision>
+        <origin xyz="0 0 0" rpy="${pi/2} 0 0" />
+        <geometry>
+          <sphere radius="${caster_radius}" />
+        </geometry>
+        <origin xyz="0 0 0" rpy="0 0 0" />
+      </collision>
+      <inertial>
+        <origin xyz="0 0 0" />
+        <mass value="0.01" />
+        <inertia ixx="0.001" ixy="0.0" ixz="0.0"
+                 iyy="0.001" iyz="0.0"
+                 izz="0.001" />
+        </inertial>
+    </link>
+    <joint name="${prefix}_caster_joint" type="fixed">
+      <axis xyz="0 1 0" rpy="0 0 0" />
+      <parent link="base_link"/>
+      <child link="${prefix}_caster"/>
+      <origin xyz="${(casterbase + caster_radius) * reflect / 2}
+                   0
+                   ${caster_offset - caster_radius}"
+              rpy="0 0 0"/>
+    </joint>
+    <gazebo reference="${prefix}_caster">
+      <mu1>0.0</mu1>
+      <mu2>0.0</mu2>
+      <kp>1000000.0</kp>
+      <kd>100.0</kd>
+      <minDepth>0.001</minDepth>
+      <maxVel>1.0</maxVel>
+      <material>Gazebo/Grey</material>
+    </gazebo>
+  </xacro:macro>
+  <xacro:caster prefix="front" reflect="1"/>
+  <xacro:caster prefix="rear" reflect="-1"/>
   <!-- Laser scanner 1D -->
   <joint name="laser_joint" type="fixed">
     <axis xyz="0 1 0" />
-    <origin xyz="0 0 ${body_height}" rpy="0 0 0"/>
+    <origin xyz="0 0 ${body_height / 2}" rpy="0 0 0"/>
     <parent link="base_link"/>
     <child link="laser_link"/>
@@ -99,5 +162,5 @@
       <origin xyz="0 0 0" rpy="0 0 0"/>
       <geometry>
-        <cylinder radius="0.05" length="0.1"/>
+        <cylinder radius="0.02" length="0.02"/>
       </geometry>
     </collision>
@@ -105,5 +168,5 @@
       <origin xyz="0 0 0" rpy="0 0 0"/>
       <geometry>
-        <cylinder radius="0.05" length="0.1"/>
+        <cylinder radius="0.02" length="0.02"/>
       </geometry>
     </visual>
@@ -111,5 +174,7 @@
       <mass value="1e-5" />
       <origin xyz="0 0 0" rpy="0 0 0"/>
-      <inertia ixx="1e-6" ixy="0" ixz="0" iyy="1e-6" iyz="0" izz="1e-6" />
+      <inertia ixx="1e-6" ixy="0" ixz="0"
+               iyy="1e-6" iyz="0"
+               izz="1e-6" />
     </inertial>
   </link>

Commit message: Add caster links to balance the wheelbase

File: goldorak_simulation/urdf/goldorak.xacro (robot description, xacro)
@@ -2,12 +2,12 @@
 <robot name="goldorak" xmlns:xacro="http://ros.org/wiki/xacro">
   <xacro:property name="body_radius" value="0.12" />
-  <xacro:property name="body_height" value="0.5" />
+  <xacro:property name="body_height" value="0.4" />
   <xacro:property name="wheelbase" value="0.194" />
   <xacro:property name="wheel_radius" value="0.029" />
   <xacro:property name="wheel_thickness" value="0.01" />
-  <xacro:property name="wheel_offset" value="-0.20" />
+  <xacro:property name="wheel_offset" value="-0.15" />
   <xacro:property name="casterbase" value="0.194" />
   <xacro:property name="caster_radius" value="0.01" />
-  <xacro:property name="caster_offset" value="-0.24" />
+  <xacro:property name="caster_offset" value="-0.19" />
   <xacro:property name="pi" value="3.1415" />
   <material name="blue">
